File: Pen-Plotter-Arduino-Shield.kicad_sch (KiCad schematic)
At the start: 41 parts, among them J1 CONN_08LOCK, J10 CONN_08LOCK, J11 CONN_04LOCK, J12 CONN_03LOCK, J13 691137710002, J14 CONN_03LOCK, J15 CONN_03LOCK, J16 CONN_03LOCK, J17 CONN_03LOCK, J18 CONN_03X2FEMALE, J19 CONN_02LOCK, J2 CONN_08LOCK, J20 CONN_02LOCK, J21 CONN_02LOCK, J22 CONN_02LOCK, J23 CONN_02LOCK, J3 CONN_02LOCK, J4 CONN_02LOCK, J5 CONN_04LOCK, J6 CONN_08LOCK, J7 CONN_08LOCK, J8 CONN_04LOCK, J9 CONN_08LOCK, U1 LM2596S-5, U2 Analog_1, U3 Analog_2, U6 Digital_1, U7 Digital_2

Commit message: update all files to Revision A
Parts:
- removed H1: MountingHole1, ArduinoMountingHoles:Arduino_MountingHole, symbol Mechanical_Arduino:MountingHole_Arduino
- removed H2: MountingHole2, ArduinoMountingHoles:Arduino_MountingHole, symbol Mechanical_Arduino:MountingHole_Arduino
- removed H3: MountingHole3, ArduinoMountingHoles:Arduino_MountingHole, symbol Mechanical_Arduino:MountingHole_Arduino
- removed H4: MountingHole4, ArduinoMountingHoles:Arduino_MountingHole, symbol Mechanical_Arduino:MountingHole_Arduino
- removed J11, J5, J8: CONN_04LOCK, Connectors:1X04_LOCK, symbol SparkFun-Connectors:CONN_04LOCK
- removed J12, J14, J15, J16, J17: CONN_03LOCK, Connectors:1X03_LOCK, symbol SparkFun-Connectors:CONN_03LOCK
- removed J13: 691137710002, FootPrints:691137710002, symbol 691137710002:691137710002
- removed J18: CONN_03X2FEMALE, Connectors:2X3, symbol SparkFun-Connectors:CONN_03X2FEMALE
- removed J3: CONN_02LOCK, Connectors:1X02_LOCK, symbol SparkFun-Connectors:CONN_02LOCK
- removed S2: TS02-66-60-BK-160-LCR-D, FootPrints:SW_TS02-66-60-BK-160-LCR-D, symbol TS02-66-60-BK-160-LCR-D:TS02-66-60-BK-160-LCR-D
- added J11, J3: Conn_01x02, Connector_JST:JST_XH_B2B-XH-A_1x02_P2.50mm_Vertical, symbol Connector_Generic:Conn_01x02
- added J12, J14, J15, J16, J24: Conn_01x04, Connector_JST:JST_XH_B4B-XH-A_1x04_P2.50mm_Vertical, symbol Connector_Generic:Conn_01x04
- added J17: TB005_-762-04BE, FootPrints:CUI_TB005 -762-04BE, symbol TB005_-762-04BE:TB005_-762-04BE
- added J18: 691137710003, FootPrints:691137710003, symbol 691137710003:691137710003
- added J25, J5, J8: Conn_01x05, Connector_JST:JST_XH_B5B-XH-A_1x05_P2.50mm_Vertical, symbol Connector_Generic:Conn_01x05
Connections:
- net 12V: now also J18.1
- net 5V: now also J12.2 (Pin_2), J14.2 (Pin_2), J15.2 (Pin_2), J16.2 (Pin_2)
- net GND: now also J11.2 (Pin_2), J12.3 (Pin_3), J14.3 (Pin_3), J15.3 (Pin_3), J16.3 (Pin_3), J18.2, J24.3 (Pin_3), J3.2 (Pin_2)
- net SERVO_PWM: now also J24.1 (Pin_1)
- net SERVO_PWR: now also J24.2 (Pin_2)
- net V_MOTOR: now also J11.1 (Pin_1), J3.1 (Pin_1)
- net X-LIMIT: now also J12.1 (Pin_1), J16.1 (Pin_1)
- net X_1: now also J25.1 (Pin_1)
- net X_2: now also J25.2 (Pin_2)
- net X_3: now also J25.3 (Pin_3)
- net X_4: now also J25.4 (Pin_4)
- net Y-LIMIT: now also J14.1 (Pin_1), J15.1 (Pin_1)
- net YL-1: now also J5.1 (Pin_1)
- net YL-2: now also J5.2 (Pin_2)
- net YL-3: now also J5.3 (Pin_3)
- net YL-4: now also J5.4 (Pin_4)
- net YR-1: now also J8.1 (Pin_1)
- net YR-2: now also J8.2 (Pin_2)
- net YR-3: now also J8.3 (Pin_3)
- net YR-4: now also J8.4 (Pin_4)
- new net GNDPWR: J12.4 (Pin_4), J14.4 (Pin_4), J15.4 (Pin_4), J16.4 (Pin_4), J17.1, J17.2, J17.3, J17.4, J18.3, J24.4 (Pin_4), J25.5 (Pin_5), J5.5 (Pin_5), J8.5 (Pin_5)
- no-connect marks 21 -> 23
Other:
- note added: "12V Fans"
- note added: "Earth Ground"
- note added: "SERVO"
- note removed: "E-STOP"
